Commit message: Add a camera on the URDF model of the robot
Add a camera and set the gravity in 'low_gravity' gazebo world

File: src/biped_robot_e3_2a_sims/urdf/biped_controled.urdf (robot description, URDF)
Before this commit: robot biped, 9 links, 8 joints
Links:
- added link camera_link, mass 1e-5; collision box size=0.05 0.05 0.05; visual box size=0.05 0.05 0.05
- link L_lowerleg_contactsensor_link: geometry collision sphere radius=0.050; visual sphere radius=0.050
- link R_lowerleg_contactsensor_link: geometry collision sphere radius=0.050; visual sphere radius=0.050
Joints:
- added joint camera_joint: type fixed, parent base, child camera_link, origin xyz=0.05 0 0 rpy=0 0 0, axis 0 1 0
